File: 7segment_counter_2digit.kicad_pcb (KiCad board)
At the start: 2 copper layers, 68.6 x 94 mm, 14 parts, among them IC1 CD4026BE, IC2 CD4026BE, SW1 SW_Reset, SW2 SW_Count, U1 5611AH, U2 2462, U3 ICM7555, U4 5611AH

Commit message: Complete PCB connections
Parts:
- moved C1 13.7 mm to (150.6, 97.8)
- moved U3 12.4 mm to (139.4, 96.5), turned to 0 degrees
Routing:
- net Net-(R2-Pad2): track 60.5 -> 31.2 mm
- net Net-(IC2-Pad10): track 0.00 -> 24.3 mm
- net Net-(C2-Pad1): track 55.3 -> 34.6 mm
- net Net-(IC1-Pad15): track 105.1 -> 114.5 mm, vias 2 -> 0
- net Net-(C1-Pad1): track 22.0 -> 15.3 mm
- added copper zone on B.Cu, net GND
- added copper zone on F.Cu, net GND
Other:
- board text added: "7 Segment Counter"
- board text added: "COUNT"
- board text added: "RESET"
- board text added: "by Sean Duffy"
- board text added: "v01"
